File: popn-keypad.kicad_sch (KiCad schematic)
At the start: 10 parts, among them U1 Arduino_Pro_Micro

Commit message: Major rewiring
I got rid of all of my ground lines in favor of a copper fill connected to ground. This made the routing my traces far less convoluted.
Connections:
- net GND: now also U1.23 (GND), U1.4 (GND)
- net S4: now also S8.1; no longer S7.1
- net S6: now also S7.1; no longer S8.1
- no-connect marks 0 -> 12
Other:
- moved on the sheet: S7, S8
Changed lines of the file:
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@@
 	(generator_version "9.0")
 	(paper "A4")
+	(junction
+		(at 181.61 66.04)
+		(diameter 0)
+		(color 0 0 0 0)
+	)
+	(no_connect
+		(at 212.09 73.66)
+	)
+	(no_connect
+		(at 212.09 66.04)
+	)
+	(no_connect
+		(at 212.09 83.82)
+	)
+	(no_connect
+		(at 212.09 86.36)
+	)
+	(no_connect
+		(at 212.09 68.58)
+	)
+	(no_connect
+		(at 212.09 60.96)
+	)
+	(no_connect
+		(at 181.61 88.9)
+	)
+	(no_connect
+		(at 212.09 78.74)
+	)
+	(no_connect
+		(at 212.09 76.2)
+	)
+	(no_connect
+		(at 212.09 71.12)
+	)
+	(no_connect
+		(at 212.09 81.28)
+	)
+	(no_connect
+		(at 212.09 88.9)
+	)
+	(wire
+		(pts
+			(xy 181.61 66.04) (xy 181.61 68.58)
+		)
+		(stroke
+			(width 0)
+			(type default)
+		)
+	)
 	(global_label "S7"
 		(shape input)
@@
 		)
 		(property "Value" "GND"
-			(at 180.3399 63.5 0)
+			(at 177.8 66.0399 90)
 			(effects
 				(font
@@
 				(path "/a278322b-c6f1-4b05-8a28-8294d8d274dd"
 					(reference "#PWR010")
+					(unit 1)
+				)
+			)
+		)
+	)
+	(symbol
+		(lib_id "power:GND")
+		(at 212.09 63.5 90)
+		(unit 1)
+		(exclude_from_sim no)
+		(in_bom yes)
+		(on_board yes)
+		(dnp no)
+		(fields_autoplaced yes)
+		(property "Reference" "#PWR011"
+			(at 218.44 63.5 0)
+			(effects
+				(font
+					(size 1.27 1.27)
+				)
+				(hide yes)
+			)
+		)
+		(property "Value" "GND"
+			(at 215.9 63.4999 90)
+			(effects
+				(font
+					(size 1.27 1.27)
+				)
+				(justify right)
+			)
+		)
+		(property "Footprint" ""
+			(at 212.09 63.5 0)
+			(effects
+				(font
+					(size 1.27 1.27)
+				)
+				(hide yes)
+			)
+		)
+		(property "Datasheet" ""
+			(at 212.09 63.5 0)
+			(effects
+				(font
+					(size 1.27 1.27)
+				)
+				(hide yes)
+			)
+		)
+		(property "Description" "Power symbol creates a global label with name \"GND\" , ground"
+			(at 212.09 63.5 0)
+			(effects
+				(font
+					(size 1.27 1.27)
+				)
+				(hide yes)
+			)
+		)
+		(pin "1"
+		)
+		(instances
+			(project "popn-keypad"
+				(path "/a278322b-c6f1-4b05-8a28-8294d8d274dd"
+					(reference "#PWR011")
 					(unit 1)
 				)
@@
 	(symbol
 		(lib_id "ScottoKeebs:Placeholder_Keyswitch")
-		(at 152.4 81.28 0)
+		(at 157.48 71.12 0)
 		(unit 1)
 		(exclude_from_sim no)
@@
 		(fields_autoplaced yes)
 		(property "Reference" "S8"
-			(at 152.4 81.28 0)
+			(at 157.48 71.12 0)
 			(do_not_autoplace yes)
 			(effects
@@
 		)
 		(property "Value" "~"
-			(at 152.4 76.2 0)
+			(at 157.48 66.04 0)
 			(effects
 				(font
@@
 		)
 		(property "Footprint" "ScottoKeebs_Hotswap:Hotswap_MX_Plated_1.00u"
-			(at 152.4 81.28 0)
-			(effects
-				(font
-					(size 1.27 1.27)
-				)
-				(hide yes)
-			)
-		)
-		(property "Datasheet" ""
-			(at 149.86 83.058 0)
+			(at 157.48 71.12 0)
+			(effects
+				(font
+					(size 1.27 1.27)
+				)
+				(hide yes)
+			)
+		)
+		(property "Datasheet" ""
+			(at 154.94 72.898 0)
 			(effects
 				(font
@@
 		)
 		(property "Description" ""
-			(at 152.4 81.28 0)
+			(at 157.48 71.12 0)
 			(effects
 				(font
@@
 	(symbol
 		(lib_id "ScottoKeebs:Placeholder_Keyswitch")
-		(at 157.48 71.12 0)
+		(at 152.4 81.28 0)
 		(unit 1)
 		(exclude_from_sim no)
@@
 		(fields_autoplaced yes)
 		(property "Reference" "S7"
-			(at 157.48 71.12 0)
+			(at 152.4 81.28 0)
 			(do_not_autoplace yes)
 			(effects
@@
 		)
 		(property "Value" "~"
-			(at 157.48 66.04 0)
+			(at 152.4 76.2 0)
 			(effects
 				(font
@@
 		)
 		(property "Footprint" "ScottoKeebs_Hotswap:Hotswap_MX_Plated_1.00u"
-			(at 157.48 71.12 0)
-			(effects
-				(font
-					(size 1.27 1.27)
-				)
-				(hide yes)
-			)
-		)
-		(property "Datasheet" ""
-			(at 154.94 72.898 0)
+			(at 152.4 81.28 0)
+			(effects
+				(font
+					(size 1.27 1.27)
+				)
+				(hide yes)
+			)
+		)
+		(property "Datasheet" ""
+			(at 149.86 83.058 0)
 			(effects
 				(font
@@
 		)
 		(property "Description" ""
-			(at 157.48 71.12 0)
-			(effects
-				(font
+			(at 152.4 81.28 0)
+			(effects
+				(font
