File: kicad/popn-keypad.kicad_sch (KiCad schematic)
At the start: 10 parts, among them U1 Arduino_Pro_Micro

Commit message: Updated to Kicad 10, renamed some parts for organization
Parts:
- S1: renamed from S2; value ~ -> (none)
- S2: renamed from S4; value ~ -> (none)
- S3: renamed from S6; value ~ -> (none)
- S4: renamed from S8; value ~ -> (none)
- S5: renamed from S9; value ~ -> (none)
- S6: renamed from S7; value ~ -> (none)
- S7: renamed from S5; value ~ -> (none)
- S8: renamed from S3; value ~ -> (none)
- S9: renamed from S1; value ~ -> (none)
